File: cad/dual_sensor_module.sch (EAGLE design)
At the start: 14 parts, among them IC1 MCP602SN, IC2 TC7660DIL8

Commit message: update pcb files
Parts:
- removed JP1, JP2: (no value), adafruit:PINHD-1X3
- added JP3, JP4: (no value), pinhead:PINHD-1X2
- added R1: (no value), rcl:R-US_R1206
- LED1: device adafruit:LEDCHIPLED_0805 -> adafruit:LED3MM
Connections:
- new net VOUT22: IC1B.OUT, R1.1, RF2.1
- net N$52: now also JP4.2; no longer JP1.3
- net N$82: now also JP3.2; no longer JP2.3
- net VOUT2: now also R1.2; no longer IC1B.OUT, RF2.1
- net VT: now also JP3.1, JP4.1; no longer JP1.1, JP2.1
Changed lines of the file:
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@@
 <?xml version="1.0" encoding="utf-8"?>
 <!DOCTYPE eagle SYSTEM "eagle.dtd">
-<eagle version="9.4.2">
+<eagle version="9.6.1">
 <drawing>
 <settings>
@@
 <part name="RF5" library="resistor" library_urn="urn:adsk.eagle:library:348" deviceset="R-US_" device="R0805" package3d_urn="urn:adsk.eagle:package:23553/2" value="10k"/>
 <part name="P+5" library="supply1" library_urn="urn:adsk.eagle:library:371" deviceset="+5V" device=""/>
-<part name="LED1" library="adafruit" deviceset="LED" device="CHIPLED_0805"/>
+<part name="LED1" library="adafruit" library_urn="urn:adsk.eagle:library:420" deviceset="LED" device="3MM" package3d_urn="urn:adsk.eagle:package:6240537/1"/>
 <part name="SUPPLY3" library="supply2" library_urn="urn:adsk.eagle:library:372" deviceset="GND" device=""/>
 <part name="R0" library="rcl" library_urn="urn:adsk.eagle:library:334" deviceset="R-US_" device="R1206" package3d_urn="urn:adsk.eagle:package:23540/2"/>
-<part name="JP1" library="adafruit" deviceset="PINHD-1X3" device=""/>
-<part name="JP2" library="adafruit" deviceset="PINHD-1X3" device=""/>
 <part name="U$1" library="robot-hand" deviceset="DYNAMIXEL_RS485" device=""/>
+<part name="R1" library="rcl" library_urn="urn:adsk.eagle:library:334" deviceset="R-US_" device="R1206" package3d_urn="urn:adsk.eagle:package:23540/2"/>
+<part name="JP3" library="pinhead" library_urn="urn:adsk.eagle:library:325" deviceset="PINHD-1X2" device="" package3d_urn="urn:adsk.eagle:package:22435/2"/>
+<part name="JP4" library="pinhead" library_urn="urn:adsk.eagle:library:325" deviceset="PINHD-1X2" device="" package3d_urn="urn:adsk.eagle:package:22435/2"/>
 </parts>
 <sheets>
@@
 <attribute name="VALUE" x="148.59" y="62.738" size="1.778" layer="96"/>
 </instance>
-<instance part="JP1" gate="A" x="109.22" y="73.66" smashed="yes" rot="R180">
-<attribute name="NAME" x="115.57" y="67.945" size="1.778" layer="95" rot="R180"/>
-<attribute name="VALUE" x="115.57" y="81.28" size="1.778" layer="96" rot="R180"/>
-</instance>
-<instance part="JP2" gate="A" x="109.22" y="35.56" smashed="yes" rot="R180">
-<attribute name="NAME" x="115.57" y="29.845" size="1.778" layer="95" rot="R180"/>
-<attribute name="VALUE" x="115.57" y="43.18" size="1.778" layer="96" rot="R180"/>
-</instance>
 <instance part="U$1" gate="J$1" x="63.5" y="38.1" smashed="yes" rot="R180">
 <attribute name="NAME" x="68.58" y="29.718" size="1.778" layer="95" rot="R180"/>
+</instance>
+<instance part="R1" gate="G$1" x="170.18" y="40.64" smashed="yes">
+<attribute name="NAME" x="166.37" y="42.1386" size="1.778" layer="95"/>
+<attribute name="VALUE" x="166.37" y="37.338" size="1.778" layer="96"/>
+</instance>
+<instance part="JP3" gate="G$1" x="109.22" y="38.1" smashed="yes" rot="R180">
+<attribute name="NAME" x="115.57" y="32.385" size="1.778" layer="95" rot="R180"/>
+<attribute name="VALUE" x="115.57" y="43.18" size="1.778" layer="96" rot="R180"/>
+</instance>
+<instance part="JP4" gate="G$1" x="109.22" y="76.2" smashed="yes" rot="R180">
+<attribute name="NAME" x="115.57" y="70.485" size="1.778" layer="95" rot="R180"/>
+<attribute name="VALUE" x="115.57" y="81.28" size="1.778" layer="96" rot="R180"/>
 </instance>
 </instances>
@@
 <pinref part="IC1" gate="B" pin="-IN"/>
 <wire x1="137.16" y1="38.1" x2="129.54" y2="38.1" width="0.1524" layer="91"/>
-<pinref part="JP2" gate="A" pin="3"/>
 <wire x1="129.54" y1="38.1" x2="111.76" y2="38.1" width="0.1524" layer="91"/>
 <junction x="129.54" y="38.1"/>
+<pinref part="JP3" gate="G$1" pin="2"/>
 </segment>
 </net>
 <net name="VOUT2" class="0">
-<segment>
-<pinref part="IC1" gate="B" pin="OUT"/>
-<pinref part="RF2" gate="G$1" pin="1"/>
-<wire x1="152.4" y1="40.64" x2="152.4" y2="27.94" width="0.1524" layer="91"/>
-<wire x1="152.4" y1="27.94" x2="147.32" y2="27.94" width="0.1524" layer="91"/>
-<wire x1="152.4" y1="40.64" x2="157.48" y2="40.64" width="0.1524" layer="91"/>
-<label x="157.48" y="40.64" size="1.778" layer="95" xref="yes"/>
-<junction x="152.4" y="40.64"/>
-</segment>
 <segment>
 <pinref part="U$1" gate="J$1" pin="D+"/>
 <wire x1="55.88" y1="38.1" x2="53.34" y2="38.1" width="0.1524" layer="91"/>
 <label x="53.34" y="38.1" size="1.778" layer="95" rot="R180" xref="yes"/>
+</segment>
+<segment>
+<pinref part="R1" gate="G$1" pin="2"/>
+<wire x1="175.26" y1="40.64" x2="182.88" y2="40.64" width="0.1524" layer="91"/>
+<label x="175.26" y="43.18" size="1.778" layer="95"/>
+<label x="180.34" y="43.18" size="1.778" layer="95" xref="yes"/>
 </segment>
 </net>
@@
 </segment>
 <segment>
-<pinref part="JP1" gate="A" pin="1"/>
-<wire x1="111.76" y1="71.12" x2="116.84" y2="71.12" width="0.1524" layer="91"/>
-<label x="116.84" y="71.12" size="1.778" layer="95" xref="yes"/>
-</segment>
-<segment>
-<pinref part="JP2" gate="A" pin="1"/>
-<wire x1="111.76" y1="33.02" x2="116.84" y2="33.02" width="0.1524" layer="91"/>
-<label x="116.84" y="33.02" size="1.778" layer="95" xref="yes"/>
+<wire x1="111.76" y1="73.66" x2="116.84" y2="73.66" width="0.1524" layer="91"/>
+<label x="116.84" y="73.66" size="1.778" layer="95" xref="yes"/>
+<pinref part="JP4" gate="G$1" pin="1"/>
+</segment>
+<segment>
+<wire x1="111.76" y1="35.56" x2="116.84" y2="35.56" width="0.1524" layer="91"/>
+<label x="116.84" y="35.56" size="1.778" layer="95" xref="yes"/>
+<pinref part="JP3" gate="G$1" pin="1"/>
 </segment>
 </net>
@@
 <wire x1="142.24" y1="60.96" x2="129.54" y2="60.96" width="0.1524" layer="91"/>
 <wire x1="129.54" y1="60.96" x2="129.54" y2="76.2" width="0.1524" layer="91"/>
-<pinref part="JP1" gate="A" pin="3"/>
 <wire x1="129.54" y1="76.2" x2="111.76" y2="76.2" width="0.1524" layer="91"/>
 <junction x="129.54" y="76.2"/>
+<pinref part="JP4" gate="G$1" pin="2"/>
 </segment>
 </net>
@@
 </segment>
 </net>
+<net name="VOUT22" class="0">
+<segment>
+<pinref part="IC1" gate="B" pin="OUT"/>
+<pinref part="RF2" gate="G$1" pin="1"/>
+<wire x1="152.4" y1="40.64" x2="152.4" y2="27.94" width="0.1524" layer="91"/>
+<wire x1="152.4" y1="27.94" x2="147.32" y2="27.94" width="0.1524" layer="91"/>
+<wire x1="152.4" y1="40.64" x2="165.1" y2="40.64" width="0.1524" layer="91"/>
+<junction x="152.4" y="40.64"/>
+<pinref part="R1" gate="G$1" pin="1"/>
+<label x="165.1" y="35.56" size="1.778" layer="95"/>
+</segment>
+</net>
